File: hardware/Nuclio-F466RE/clearair.kicad_sch (KiCad schematic)
At the start: 33 parts, among them J1 220VAC mains in, M1 AC vent fan, Q1 2N7000, Q2 2N7000, Q3 2N2222A, Q4 IRFZ44N, SW1 RESET, SW2 COLD_BOOT, U1 SPS30, U2 BME680, U3 MQ131, U4 MiCS-4514, U5 RobotDyn AC dimmer

Commit message: add kicad schema
Parts:
- added JP1: FAN_V_SEL, symbol Jumper:Jumper_3_Open
- added M2: 40mm fan (5V or 12V), symbol Motor:Fan
Connections:
- net +12V: now also JP1.3 (B)
- net +5V: now also JP1.1 (A)
- net GND: now also SW1.1, SW2.1, M2.2 (-); no longer SW1.2, SW2.2
- net AC_L: no longer names the net of J1.1 (Pin_1), PS1.1 (Pin_1), U5.5 (IN)
- net AC_N: no longer names the net of J1.2 (Pin_2), M1.2, PS1.2 (Pin_2), U5.6 (N)
- net BOOT_TY_SELECT: no longer names the net of A1.3 (PC12)
- net BOOT_TY_SELECT: now also SW2.2; no longer SW2.1
- net BUZZER_B: no longer names the net of Q3.2 (B), R9.2
- net BUZZER_GATE: no longer names the net of Q3.3 (C), Q4.1 (G), R16.2
- net BUZZER_N: no longer names the net of BZ1.2 (-), Q4.2 (D)
- net DIMMER_LEVEL: no longer names the net of A1.57 (PC7), U5.4 (PSM)
- net FAN_OUT: no longer names the net of M1.1, U5.7 (OUT)
- net I2C3_SCL: no longer names the net of A1.61 (PA8), R1.2, U1.3 (SCL), U2.3 (SCL)
- net I2C3_SDA: no longer names the net of A1.39 (PC9), R2.2, U1.2 (SDA), U2.4 (SDA)
- net MICS4514_CO: no longer names the net of A1.30 (PA1), R6.1
- net MICS4514_CO: now also R5.1; no longer R5.2
- net MICS4514_NO2: no longer names the net of A1.53 (PA7), R7.2, R8.1
- net MICS4514_PREHEAT: no longer names the net of A1.40 (PC8), U4.5 (PRE)
- net MICS_NOX: no longer names the net of R7.1, U4.4 (NOX)
- net MICS_RED: no longer names the net of U4.3 (RED)
- net MICS_RED: now also R5.2; no longer R5.1
- net MQ131_AO: no longer names the net of R3.1, U3.4 (AO)
- net MQ131_READ: no longer names the net of A1.28 (PA0), R3.2, R4.1
- net NANO_RX: no longer names the net of A2.2 (D0/RX), Q1.3 (D), R11.2
- net NANO_TX: no longer names the net of A2.1 (D1/TX), Q2.3 (D), R13.2
- net NRST: no longer names the net of A1.14 (RESET)
- net NRST: now also SW1.2; no longer SW1.1
- net USART3_RX: no longer names the net of A1.44 (PC5), Q2.1 (S), R12.2
- net USART3_TX: no longer names the net of A1.63 (PB10), Q1.1 (S), R10.2
- net ZC_5V: no longer names the net of R14.1
- net ZC_5V: now also A1.42 (PC6), R15.1; no longer U5.3 (Z-C)
- removed net ZC_INPUT: A1.42 (PC6), R14.2, R15.1
- new net: JP1.2 (C), M2.1 (+)
- new net: R14.2, U5.3 (Z-C)
Other:
- note added: "220VAC mains split: J1 -> RobotDyn TRIAC (fan) and PS1 AC-DC (12V buzzer, 5V board + peripherals). PS1 pins: 1 L, 2 N, 3 +12V, 4 +5V, 5 GND. USART3 (future Arduino link): PB10 TX / PC5 RX."
- note added: "5V outputs -> 1k8 (series) / 3k3 (to GND) divider -> 3.24V max at MCU pin: MQ131 AO -> PA0, MiCS RED -> PA1, MiCS NOX -> PA7, RobotDyn Z-C -> PC6."
- note added: "Buzzer: R9 input left floating (GPIO not assigned in clearair.ioc). Q3 inverts: input HIGH -> buzzer OFF; LOW/floating -> R16 pulls IRFZ44N gate to 12V -> buzzer ON."
- note added: "HIGH VOLTAGE: J1, PS1 pins 1-2, RobotDyn IN/N/OUT, M1 carry 220VAC."
- note added: "I2C3: SPS30 SEL=GND (I2C, 0x69); BME680 SDO=3V3 (0x77), CS=3V3. 4k7 pull-ups to 3V3."
- note added: "M2 40mm fan runs all the time. JP1: bridge 1-2 for a 5V fan, 2-3 for a 12V fan."
- note added: "NUCLEO-F446RE: JP5 on E5V, 5V from PS1 into CN7-6. 3V3 from on-board regulator (CN7-16). On-board only: PA2/PA3 ST-LINK VCP, PA5 LD2, PC13 B1, PA13/PA14 SWD, PH0/PH1 HSE, PC14/PC15 LSE."
- note removed: "AC phase control - RobotDyn TRIAC dimmer (HIGH VOLTAGE side right of module)"
- note removed: "Analog gas sensors (5V outputs divided to <3.3V for ADC)"
- note removed: "Divider 1k8 (top) / 3k3 (to GND): 5V -> 3.24V max at ADC pin. MQ131 DO unused. MiCS PRE driven HIGH by PC8 during heater warm-up."
- note removed: "I2C3 sensors (3V3 pull-ups)"
- note removed: "MCU - NUCLEO-F446RE (ST morpho CN7 / CN10)"
- note removed: "Manual controls"
- note removed: "Module VCC = 5V. Z-C (5V) -> 1k8/3k3 divider -> PC6 (EXTI6). PSM <- PC7 gate pulse from TIM3 ISR. AC_L / AC_N from J1 mains."
- note removed: "Nano D2..D13 / A0..A7 drive the future LED array / 7-seg display and 2 boot-mode LEDs (not defined yet)."
- note removed: "No PWR_FLAG on +5V / +3V3: Nucleo +3V3 and Nano +5V pins are power outputs in their symbols. Real 5V source: PS1."
- note removed: "On-board only (no external wire): PA2/PA3 USART2 = ST-LINK VCP, PA5 = LD2, PC13 = B1, PA13/PA14 = SWD, PH0/PH1 = HSE (ST-LINK MCO), PC14/PC15 = LSE. Power: JP5 on E5V, external 5V on CN7-6."
- note removed: "PS1: 1 AC L 2 AC N 3 +12V (buzzer) 4 +5V (Nucleo E5V + peripherals) 5 GND 3V3 comes from the Nucleo on-board regulator (CN7-16)."
- note removed: "Power - 220VAC mains split to TRIAC dimmer and AC-DC PSU"
- note removed: "R9 pin 1 = buzzer control input, left floating (GPIO not assigned in clearair.ioc). Q3 is an inverting stage: R9 input HIGH -> Q3 on -> gate LOW -> buzzer OFF; input LOW / floating -> R16 pulls gate to 12V -> buzzer ON. Verify polarity vs firmware."
- note removed: "SDO = 3V3: addr 0x77 (BME68X_I2C_ADDR_HIGH) CS = 3V3: I2C mode"
- note removed: "SEL = GND: I2C mode, addr 0x69"
- note removed: "SW1 parallel to Nucleo B2 (NRST). SW2: PC12 internal pull-up, read once at boot."
- note removed: "Safety-latch buzzer (12V) - 2N2222A drives IRFZ44N low-side switch"
- note removed: "USART3 link to Arduino Nano (future) - 2N7000 3V3<->5V level shift"
