File: hardware/WeAct-G474CE-Long/clearair.kicad_sch (KiCad schematic)
At the start: 36 parts, among them J1 220VAC mains in, M1 AC vent fan, M2 40mm fan (5V or 12V), Q1 2N7000, Q2 2N7000, Q3 2N2222A, Q4 IRFZ44N, SW1 RESET, SW2 COLD_BOOT, U1 SPS30, U2 BME680, U3 MQ131, U4 MiCS-4514, U5 RobotDyn AC dimmer

Commit message: chenge pin PB12 perpose
Parts:
- added U6: PCF8563 RTC, libraries:PCF8563_HW689, symbol FullModules:PCF8563_HW689
Connections:
- net +3V3: now also U6.1 (VCC)
- net GND: now also U6.2 (GND)
- net at A.10 (PA15), R1.2, U1.3 (SCL)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: now also U6.4 (SCL)
- net at A.3 (PB7), R2.2, U1.2 (SDA)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: now also U6.3 (SDA)
- no-connect marks 53 -> 55
Other:
- note added: "I2C1: PA15 SCL / PB7 SDA. SPS30 SEL=GND (I2C, 0x69); BME680 SDO=3V3 (0x77), CS=3V3; PCF8563 RTC HW-689 (0x51, CR1220, COT and INT unused). 4k7 pull-ups to 3V3."
- note removed: "I2C1: PA15 SCL / PB7 SDA. SPS30 SEL=GND (I2C, 0x69); BME680 SDO=3V3 (0x77), CS=3V3. 4k7 pull-ups to 3V3."
Changed lines of the file:
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@@
 	(no_connect (at 477.52 208.28))
 	(text "WeAct STM32G474CEU6 Long (A1): 5V from PS1 into P3 VDD5V (pins 43/44). 3V3 from the on-board LDO (P4 pins 47/48, P5 pin 52).\nPin map: clear-air.ioc + README \"STM32G474CEU6 Pin Plan\". On-board only: PC6 user LED (LED_BOARD), PC13 user key, PB8 BOOT0 key,\nPA11/PA12 USB-C, PF0/PF1 8 MHz HSE, PC14/PC15 LSE. VREF+ (pin 37) tied to 3V3 so the ADCs read against 3.3V." (exclude_from_sim no) (at 25.4 335.28 0) (effects (font (size 1.27 1.27)) (justify left top)))
-	(text "I2C1: PA15 SCL / PB7 SDA. SPS30 SEL=GND (I2C, 0x69); BME680 SDO=3V3 (0x77), CS=3V3. 4k7 pull-ups to 3V3." (exclude_from_sim no) (at 25.4 345.44 0) (effects (font (size 1.27 1.27)) (justify left top)))
+	(text "I2C1: PA15 SCL / PB7 SDA. SPS30 SEL=GND (I2C, 0x69); BME680 SDO=3V3 (0x77), CS=3V3; PCF8563 RTC HW-689 (0x51, CR1220, COT and INT unused). 4k7 pull-ups to 3V3." (exclude_from_sim no) (at 25.4 345.44 0) (effects (font (size 1.27 1.27)) (justify left top)))
 	(text "5V outputs -> 1k8 (series) / 3k3 (to GND) divider -> 3.24V max at MCU pin:\nMQ131 AO -> PA0 (ADC1_IN1), MiCS RED -> PA1 (ADC2_IN2), MiCS NOX -> PA7 (ADC2_IN4), RobotDyn Z-C -> PB0 (EXTI0)." (exclude_from_sim no) (at 25.4 350.52 0) (effects (font (size 1.27 1.27)) (justify left top)))
 	(text "Buzzer: PB15 (BUZZER_IN) -> R9 -> Q3. Q3 inverts: PB15 HIGH -> buzzer OFF; LOW -> R16 pulls IRFZ44N gate to 12V -> buzzer ON.\nMiCS-4514 PRE <- PB12 (MICS_PREHEAT). Cold/warm boot button SW2 -> PB14 (BOOT_MODE, pull-up). Gate PB1 (TRIAC_DIMMER) -> RobotDyn PSM." (exclude_from_sim no) (at 25.4 358.14 0) (effects (font (size 1.27 1.27)) (justify left top)))
@@
 	(text "220VAC mains split: J1 -> RobotDyn TRIAC (fan) and PS1 AC-DC (12V buzzer, 5V board + peripherals).\nPS1 pins: 1 L, 2 N, 3 +12V, 4 +5V, 5 GND. M2 40mm fan runs all the time. JP1: bridge 1-2 for a 5V fan, 2-3 for a 12V fan." (exclude_from_sim no) (at 25.4 375.92 0) (effects (font (size 1.27 1.27)) (justify left top)))
 	(text "HIGH VOLTAGE: J1, PS1 pins 1-2, RobotDyn IN/N/OUT, M1 carry 220VAC." (exclude_from_sim no) (at 420 25.4 0) (effects (font (size 1.27 1.27)) (justify left top)))
+	(symbol (lib_id "FullModules:PCF8563_HW689") (at 238.76 199.39 270) (unit 1)
+		(exclude_from_sim no) (in_bom yes) (on_board yes) (dnp no)
+		(property "Reference" "U6" (at 241.3 187.96 90) (effects (font (size 1.27 1.27))))
+		(property "Value" "PCF8563 RTC" (at 241.3 211.0 90) (effects (font (size 1.27 1.27))))
+		(property "Footprint" "libraries:PCF8563_HW689" (at 238.76 199.39 90) (effects (font (size 1.27 1.27)) (hide yes)))
+		(property "Datasheet" "https://www.nxp.com/docs/en/data-sheet/PCF8563.pdf" (at 238.76 199.39 90) (effects (font (size 1.27 1.27)) (hide yes)))
+		(property "Description" "PCF8563 real-time clock module, board marking HW-689 (43 x 17 mm), I2C address 0x51, 1.0-5.5 V. 6-pin header VCC/GND/SDA/SCL/COT/INT in the order printed on the board. COT is the programmable clock output, INT is the open-drain alarm/timer interrupt (needs a pull-up if used). CR1220 backup cell holder on board (12.5 mm cell, 3.5 mm deep). The photographed board seems to have no I2C pull-ups: add 4.7k to 3V3 on the bus." (at 238.76 199.39 90) (effects (font (size 1.27 1.27)) (hide yes)))
+		(property "ki_keywords" "PCF8563 HW-689 RTC real time clock I2C module CR1220" (at 238.76 199.39 90) (effects (font (size 1.27 1.27)) (hide yes)))
+		(pin "1")
+		(pin "2")
+		(pin "3")
+		(pin "4")
+		(pin "5")
+		(pin "6")
+		(instances (project "clearair" (path "/953560a5-36cf-5251-8f8d-509802d70a69" (reference "U6") (unit 1)))))
+	(wire (pts (xy 233.68 193.04) (xy 220.98 193.04)) (stroke (width 0) (type default)))
+	(junction (at 220.98 193.04) (diameter 0) (color 0 0 0 0))
+	(wire (pts (xy 233.68 195.58) (xy 231.14 195.58)) (stroke (width 0) (type default)))
+	(junction (at 231.14 195.58) (diameter 0) (color 0 0 0 0))
+	(wire (pts (xy 233.68 198.12) (xy 226.06 198.12)) (stroke (width 0) (type default)))
+	(junction (at 226.06 198.12) (diameter 0) (color 0 0 0 0))
+	(wire (pts (xy 233.68 200.66) (xy 223.52 200.66)) (stroke (width 0) (type default)))
+	(junction (at 223.52 200.66) (diameter 0) (color 0 0 0 0))
+	(no_connect (at 233.68 203.2))
+	(no_connect (at 233.68 205.74))
 	(sheet_instances (path "/" (page "1")))
 	(embedded_fonts no)

Commit message: change pin PB12 purpose to serv prehead of MQ131
Parts:
- added Q5: AO3400A, Package_TO_SOT_SMD:SOT-23, symbol Transistor_FET:AO3400A
- added R17: 100, symbol Device:R
- added R18: 100k, symbol Device:R
Connections:
- net GND: now also U4.5 (PRE), Q5.2 (S), R18.2; no longer U3.2 (GND)
- net at A.20 (PB12): now also R17.1; no longer U4.5 (PRE)
- new net: Q5.1 (G), R17.2, R18.1
- new net: Q5.3 (D), U3.2 (GND)
Other:
- note added: "Buzzer: PB15 (BUZZER_IN) -> R9 -> Q3. Q3 inverts: PB15 HIGH -> buzzer OFF; LOW -> R16 pulls IRFZ44N gate to 12V -> buzzer ON. MiCS-4514 PRE tied to GND (boost not used). PB12 (MQ131_PREHEAT) -> R17 100R -> Q5 AO3400A gate, R18 100k pull-down: low-side switch in the MQ131 GND, HIGH = heater on. Cold/warm boot button SW2 -> PB14 (BOOT_MODE, pull-up). Gate PB1 (TRIAC_DIMMER) -> RobotDyn PSM."
- note removed: "Buzzer: PB15 (BUZZER_IN) -> R9 -> Q3. Q3 inverts: PB15 HIGH -> buzzer OFF; LOW -> R16 pulls IRFZ44N gate to 12V -> buzzer ON. MiCS-4514 PRE <- PB12 (MICS_PREHEAT). Cold/warm boot button SW2 -> PB14 (BOOT_MODE, pull-up). Gate PB1 (TRIAC_DIMMER) -> RobotDyn PSM."
Changed lines of the file:
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@@
 	(wire (pts (xy 276.86 224.79) (xy 276.86 215.9)) (stroke (width 0) (type default)))
 	(wire (pts (xy 276.86 215.9) (xy 281.94 215.9)) (stroke (width 0) (type default)))
-	(wire (pts (xy 294.64 299.72) (xy 281.94 299.72)) (stroke (width 0) (type default)))
 	(wire (pts (xy 281.94 299.72) (xy 281.94 223.52)) (stroke (width 0) (type default)))
 	(wire (pts (xy 177.8 76.2) (xy 173.99 76.2)) (stroke (width 0) (type default)))
@@
 	(wire (pts (xy 367.03 179.07) (xy 367.03 160.02)) (stroke (width 0) (type default)))
 	(wire (pts (xy 367.03 160.02) (xy 345.44 160.02)) (stroke (width 0) (type default)))
-	(wire (pts (xy 391.16 180.34) (xy 391.16 179.07)) (stroke (width 0) (type default)))
-	(wire (pts (xy 391.16 179.07) (xy 367.03 179.07)) (stroke (width 0) (type default)))
 	(wire (pts (xy 355.6 232.41) (xy 355.6 233.68)) (stroke (width 0) (type default)))
 	(wire (pts (xy 355.6 233.68) (xy 363.22 233.68)) (stroke (width 0) (type default)))
@@
 	(junction (at 318.77 175.26) (diameter 0) (color 0 0 0 0))
 	(junction (at 363.22 201.93) (diameter 0) (color 0 0 0 0))
-	(junction (at 367.03 179.07) (diameter 0) (color 0 0 0 0))
 	(junction (at 355.6 233.68) (diameter 0) (color 0 0 0 0))
 	(junction (at 363.22 233.68) (diameter 0) (color 0 0 0 0))
@@
 	(text "I2C1: PA15 SCL / PB7 SDA. SPS30 SEL=GND (I2C, 0x69); BME680 SDO=3V3 (0x77), CS=3V3; PCF8563 RTC HW-689 (0x51, CR1220, COT and INT unused). 4k7 pull-ups to 3V3." (exclude_from_sim no) (at 25.4 345.44 0) (effects (font (size 1.27 1.27)) (justify left top)))
 	(text "5V outputs -> 1k8 (series) / 3k3 (to GND) divider -> 3.24V max at MCU pin:\nMQ131 AO -> PA0 (ADC1_IN1), MiCS RED -> PA1 (ADC2_IN2), MiCS NOX -> PA7 (ADC2_IN4), RobotDyn Z-C -> PB0 (EXTI0)." (exclude_from_sim no) (at 25.4 350.52 0) (effects (font (size 1.27 1.27)) (justify left top)))
-	(text "Buzzer: PB15 (BUZZER_IN) -> R9 -> Q3. Q3 inverts: PB15 HIGH -> buzzer OFF; LOW -> R16 pulls IRFZ44N gate to 12V -> buzzer ON.\nMiCS-4514 PRE <- PB12 (MICS_PREHEAT). Cold/warm boot button SW2 -> PB14 (BOOT_MODE, pull-up). Gate PB1 (TRIAC_DIMMER) -> RobotDyn PSM." (exclude_from_sim no) (at 25.4 358.14 0) (effects (font (size 1.27 1.27)) (justify left top)))
+	(text "Buzzer: PB15 (BUZZER_IN) -> R9 -> Q3. Q3 inverts: PB15 HIGH -> buzzer OFF; LOW -> R16 pulls IRFZ44N gate to 12V -> buzzer ON.\nMiCS-4514 PRE tied to GND (boost not used). PB12 (MQ131_PREHEAT) -> R17 100R -> Q5 AO3400A gate, R18 100k pull-down: low-side switch in the MQ131 GND, HIGH = heater on. Cold/warm boot button SW2 -> PB14 (BOOT_MODE, pull-up). Gate PB1 (TRIAC_DIMMER) -> RobotDyn PSM." (exclude_from_sim no) (at 25.4 358.14 0) (effects (font (size 1.27 1.27)) (justify left top)))
 	(text "J2 = STLINK-V3MINIE STDC14: 3 T_VCC, 4 SWDIO, 5/7/11 GND, 6 SWCLK, 12 T_NRST, 13 T_VCP_RX, 14 T_VCP_TX; 1/2/8/9/10 unused.\nSWD goes to the board P5 header (SWCLK/SWDIO/3V3/GND). USART2 VCP: PA2 TX -> T_VCP_TX, PA3 RX <- T_VCP_RX.\nUSART3 (future Arduino link): PB10 TX / PB11 RX through 2N7000 level shifters Q1/Q2." (exclude_from_sim no) (at 25.4 365.76 0) (effects (font (size 1.27 1.27)) (justify left top)))
 	(text "220VAC mains split: J1 -> RobotDyn TRIAC (fan) and PS1 AC-DC (12V buzzer, 5V board + peripherals).\nPS1 pins: 1 L, 2 N, 3 +12V, 4 +5V, 5 GND. M2 40mm fan runs all the time. JP1: bridge 1-2 for a 5V fan, 2-3 for a 12V fan." (exclude_from_sim no) (at 25.4 375.92 0) (effects (font (size 1.27 1.27)) (justify left top)))
@@
 	(no_connect (at 233.68 203.2))
 	(no_connect (at 233.68 205.74))
+	(symbol (lib_id "Transistor_FET:AO3400A") (at 393.7 207.01 0) (unit 1)
+		(exclude_from_sim no) (in_bom yes) (on_board yes) (dnp no)
+		(property "Reference" "Q5" (at 399.288 202.565 0) (effects (font (size 1.27 1.27)) (justify left)))
+		(property "Value" "AO3400A" (at 401.955 208.915 90) (effects (font (size 1.27 1.27))))
+		(property "Footprint" "Package_TO_SOT_SMD:SOT-23" (at 398.78 208.915 0) (effects (font (size 1.27 1.27)) (hide yes)))
+		(property "Datasheet" "http://www.aosmd.com/pdfs/datasheet/AO3400A.pdf" (at 393.7 207.01 0) (effects (font (size 1.27 1.27)) (hide yes)))
+		(property "Description" "30V Vds, 5.7A Id, N-Channel MOSFET, SOT-23. Low-side switch in the MQ131 module GND: PB12 HIGH = heater on." (at 393.7 207.01 0) (effects (font (size 1.27 1.27)) (hide yes)))
+		(property "ki_keywords" "N-Channel MOSFET" (at 393.7 207.01 0) (effects (font (size 1.27 1.27)) (hide yes)))
+		(property "ki_fp_filters" "SOT?23*" (at 393.7 207.01 0) (effects (font (size 1.27 1.27)) (hide yes)))
+		(pin "1")
+		(pin "2")
+		(pin "3")
+		(instances (project "clearair" (path "/953560a5-36cf-5251-8f8d-509802d70a69" (reference "Q5") (unit 1)))))
+	(symbol (lib_id "Device:R") (at 381.0 207.01 90) (unit 1)
+		(exclude_from_sim no) (in_bom yes) (on_board yes) (dnp no)
+		(property "Reference" "R17" (at 381.0 204.47 0) (effects (font (size 1.27 1.27))))
+		(property "Value" "100" (at 381.0 209.55 0) (effects (font (size 1.27 1.27))))
+		(property "Footprint" "" (at 381.0 207.01 0) (effects (font (size 1.27 1.27)) (hide yes)))
+		(property "Datasheet" "" (at 381.0 207.01 0) (effects (font (size 1.27 1.27)) (hide yes)))
+		(property "Description" "Resistor" (at 381.0 207.01 0) (effects (font (size 1.27 1.27)) (hide yes)))
+		(property "ki_keywords" "R res resistor" (at 381.0 207.01 0) (effects (font (size 1.27 1.27)) (hide yes)))
+		(property "ki_fp_filters" "R_*" (at 381.0 207.01 0) (effects (font (size 1.27 1.27)) (hide yes)))
+		(pin "1")
+		(pin "2")
+		(instances (project "clearair" (path "/953560a5-36cf-5251-8f8d-509802d70a69" (reference "R17") (unit 1)))))
+	(symbol (lib_id "Device:R") (at 388.62 212.09 0) (unit 1)
+		(exclude_from_sim no) (in_bom yes) (on_board yes) (dnp no)
+		(property "Reference" "R18" (at 390.652 212.09 90) (effects (font (size 1.27 1.27))))
+		(property "Value" "100k" (at 388.62 212.09 90) (effects (font (size 1.27 1.27))))
+		(property "Footprint" "" (at 388.62 212.09 90) (effects (font (size 1.27 1.27)) (hide yes)))
+		(property "Datasheet" "" (at 388.62 212.09 0) (effects (font (size 1.27 1.27)) (hide yes)))
+		(property "Description" "Resistor" (at 388.62 212.09 0) (effects (font (size 1.27 1.27)) (hide yes)))
+		(property "ki_keywords" "R res resistor" (at 388.62 212.09 0) (effects (font (size 1.27 1.27)) (hide yes)))
+		(property "ki_fp_filters" "R_*" (at 388.62 212.09 0) (effects (font (size 1.27 1.27)) (hide yes)))
+		(pin "1")
+		(pin "2")
+		(instances (project "clearair" (path "/953560a5-36cf-5251-8f8d-509802d70a69" (reference "R18") (unit 1)))))
+	(wire (pts (xy 294.64 299.72) (xy 294.64 294.64)) (stroke (width 0) (type default)))
+	(wire (pts (xy 294.64 294.64) (xy 302.26 294.64)) (stroke (width 0) (type default)))
+	(wire (pts (xy 281.94 299.72) (xy 281.94 320.04)) (stroke (width 0) (type default)))
+	(wire (pts (xy 281.94 320.04) (xy 377.19 320.04)) (stroke (width 0) (type default)))
+	(wire (pts (xy 377.19 320.04) (xy 377.19 207.01)) (stroke (width 0) (type default)))
+	(wire (pts (xy 384.81 207.01) (xy 388.62 207.01)) (stroke (width 0) (type default)))
+	(wire (pts (xy 388.62 207.01) (xy 388.62 208.28)) (stroke (width 0) (type default)))
+	(wire (pts (xy 388.62 215.9) (xy 396.24 215.9)) (stroke (width 0) (type default)))
+	(wire (pts (xy 396.24 215.9) (xy 396.24 212.09)) (stroke (width 0) (type default)))
+	(wire (pts (xy 388.62 215.9) (xy 367.03 215.9)) (stroke (width 0) (type default)))
+	(wire (pts (xy 367.03 215.9) (xy 367.03 201.93)) (stroke (width 0) (type default)))
+	(wire (pts (xy 391.16 180.34) (xy 388.62 180.34)) (stroke (width 0) (type default)))
+	(wire (pts (xy 388.62 180.34) (xy 388.62 199.39)) (stroke (width 0) (type default)))
+	(wire (pts (xy 388.62 199.39) (xy 396.24 199.39)) (stroke (width 0) (type default)))
+	(wire (pts (xy 396.24 199.39) (xy 396.24 201.93)) (stroke (width 0) (type default)))
+	(junction (at 302.26 294.64) (diameter 0) (color 0 0 0 0))
+	(junction (at 388.62 207.01) (diameter 0) (color 0 0 0 0))
+	(junction (at 388.62 215.9) (diameter 0) (color 0 0 0 0))
+	(junction (at 367.03 201.93) (diameter 0) (color 0 0 0 0))
 	(sheet_instances (path "/" (page "1")))
 	(embedded_fonts no)
