File: hardware/WeAct-G474CE-Long/clearair.kicad_sch (KiCad schematic)
At the start: 40 parts, among them J1 220VAC mains in, J2 STLINK-V3MINIE STDC14, J3 SPS30, J4 BME680, J5 MQ131, J6 MiCS-4514, J7 RTC PCF8563, J8 Arduino, M1 AC vent fan, M2 80mm fan front, M3 80mm fan rear, Q1 2N7000, Q2 2N7000, Q3 2N2222A, SW1 RESET red, SW2 COLD_BOOT white, U5 RobotDyn AC dimmer

Commit message: add missing J8
Parts:
- Q1, Q2, R10, R11, R12, R13: Optional Arduino display link, future -> (none)
Changed lines of the file:
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@@
-			)
-		)
-		(property "Optional" "Arduino display link, future"
-			(at 406.4 205.74 0)
-			(hide yes)
-			(show_name no)
-			(do_not_autoplace no)
-			(effects
-				(font
-					(size 1.27 1.27)
-				)
 			)
 		)
@@
 			)
 		)
-		(property "Optional" "Arduino display link, future"
-			(at 419.1 243.84 0)
-			(hide yes)
-			(show_name no)
-			(do_not_autoplace no)
-			(effects
-				(font
-					(size 1.27 1.27)
-				)
-			)
-		)
 		(pin "1"
 		)
@@
 			)
 		)
-		(property "Optional" "Arduino display link, future"
-			(at 431.8 205.74 0)
-			(hide yes)
-			(show_name no)
-			(do_not_autoplace no)
-			(effects
-				(font
-					(size 1.27 1.27)
-				)
-			)
-		)
 		(pin "1"
 		)
@@
 			)
 		)
-		(property "Optional" "Arduino display link, future"
-			(at 406.4 233.68 0)
-			(hide yes)
-			(show_name no)
-			(do_not_autoplace no)
-			(effects
-				(font
-					(size 1.27 1.27)
-				)
-			)
-		)
 		(pin "1"
 		)
@@
 			)
 		)
-		(property "Optional" "Arduino display link, future"
-			(at 419.1 215.9 0)
-			(hide yes)
-			(show_name no)
-			(do_not_autoplace no)
-			(effects
-				(font
-					(size 1.27 1.27)
-				)
-			)
-		)
 		(pin "1"
 		)
@@
 			(at 431.8 233.68 0)
 			(hide yes)
-			(show_name no)
-			(do_not_autoplace no)
-			(effects
-				(font
-					(size 1.27 1.27)
-				)
-			)
-		)
-		(property "Optional" "Arduino display link, future"
-			(at 431.8 233.68 0)
-			(hide yes)

Commit message: add wire colors (8)
Parts:
- J4: Tie high (none) -> 5 6
- M1: Wire colors (none) -> +12V:red;+5V:red;+3V3:red;GND:black;Buzzer GND:black;Buzzer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
Changed lines of the file:
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@@
+			)
+		)
+		(property "Tie high" "5 6"
+			(at 0 0 0)
+			(hide yes)
+			(show_name no)
+			(do_not_autoplace no)
+			(effects
+				(font
+					(size 1.27 1.27)
+				)
 			)
 		)
@@
 			(hide yes)
 			(show_name no)
+			(do_not_autoplace no)
+			(effects
+				(font
+					(size 1.27 1.27)
+				)
+			)
+		)
+		(property "Wire colors" "+12V:red;+5V:red;+3V3:red;GND:black;Buzzer GND:black;Buzzer base:orange;Buzzer drive:orange;MQ131 out:yellow;MiCS CO:yellow;MiCS NO2:yellow;Front fan PWM:yellow;Rear fan PWM:yellow;I2C SCL:green;I2C SDA:blue;Front fan tach:grey;Rear fan tach:grey;ZC in:orange;ZC out:orange;TRIAC gate:orange;Reset button:orange;Cold-boot button:orange;Display TX:purple;Display RX:purple"
+			(at 0 0 0)
+			(hide yes)
+			(show_name no)

Commit message: make kicad standard, make wire_list.py a generic script
Parts:
- A1: Role mcu female -> (none)
- BZ1, M2, M3: Role heavy -> (none)
- J3, J5, J6: Role sensor -> (none)
- J4: symbol Connector_Generic:Conn_01x06 -> clearair:BME680_Header; Tie high 5 6 -> (none)
- M1: Role heavy -> (none); Wire colors +12V:red;+5V:red;+3V3:red;GND:black;Buzzer GND:black;Buzzer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 -> (none)
- PS1: Role post heavy -> (none)
- R1, R2: Bus area A14:Q18 -> (none); Role bus -> (none)
- U5: Role header -> (none)
Changed lines of the file:
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@@
 			)
 		)
-		(property "Role" "sensor"
-			(at 299.72 304.8 0)
-			(hide yes)
-			(show_name no)
-			(do_not_autoplace no)
-			(effects
-				(font
-					(size 1.27 1.27)
-				)
-			)
-		)
 		(property "Net Pin_3" "MiCS CO"
 			(at 299.72 304.8 0)
@@
 	)
 	(symbol
-		(lib_id "Connector_Generic:Conn_01x06")
+		(lib_id "clearair:BME680_Header")
 		(at 215.9 214.63 180)
 		(unit 1)
@@
 			)
 		)
-		(property "Tie high" "5 6"
-			(at 0 0 0)
-			(hide yes)
-			(show_name no)
-			(do_not_autoplace no)
-			(effects
-				(font
-					(size 1.27 1.27)
-				)
-			)
-		)
 		(pin "1"
 		)
@@
 			)
 		)
-		(property "Role" "heavy"
-			(at 510.54 66.04 0)
-			(hide yes)
-			(show_name no)
-			(do_not_autoplace no)
-			(effects
-				(font
-					(size 1.27 1.27)
-				)
-			)
-		)
-		(property "Wire colors" "+12V:red;+5V:red;+3V3:red;GND:black;Buzzer GND:black;Buzzer base:orange;Buzzer drive:orange;MQ131 out:yellow;MiCS CO:yellow;MiCS NO2:yellow;Front fan PWM:yellow;Rear fan PWM:yellow;I2C SCL:green;I2C SDA:blue;Front fan tach:grey;Rear fan tach:grey;ZC in:orange;ZC out:orange;TRIAC gate:orange;Reset button:orange;Cold-boot button:orange;Display TX:purple;Display RX:purple"
-			(at 0 0 0)
-			(hide yes)
-			(show_name no)
-			(do_not_autoplace no)
-			(effects
-				(font
-					(size 1.27 1.27)
-				)
-			)
-		)
 		(pin "1"
 		)
@@
 			)
 		)
-		(property "Role" "mcu female"
-			(at 299.72 200.66 0)
-			(hide yes)
-			(show_name no)
-			(do_not_autoplace no)
-			(effects
-				(font
-					(size 1.27 1.27)
-				)
-			)
-		)
 		(property "Net PA0" "MQ131 out"
 			(at 299.72 200.66 0)
@@
 			)
 		)
-		(property "Role" "sensor"
-			(at 215.9 180.34 0)
-			(hide yes)
-			(show_name no)
-			(do_not_autoplace no)
-			(effects
-				(font
-					(size 1.27 1.27)
-				)
-			)
-		)
 		(pin "1"
 		)
@@
 			)
 		)
-		(property "Role" "heavy"
-			(at 213.36 63.5 0)
-			(hide yes)
-			(show_name no)
-			(do_not_autoplace no)
-			(effects
-				(font
-					(size 1.27 1.27)
-				)
-			)
-		)
 		(property "Net -" "Buzzer GND"
 			(at 213.36 63.5 0)
@@
 			)
 		)
-		(property "Role" "heavy"
-			(at 288.29 76.2 0)
-			(hide yes)
-			(show_name no)
-			(do_not_autoplace no)
-			(effects
-				(font
-					(size 1.27 1.27)
-				)
-			)
-		)
 		(property "Net Pin_4" "Rear fan PWM"
 			(at 288.29 76.2 0)
@@
 			)
 		)
-		(property "Role" "header"
-			(at 457.2 66.04 0)
-			(hide yes)
-			(show_name no)
-			(do_not_autoplace no)
-			(effects
-				(font
-					(size 1.27 1.27)
-				)
-			)
-		)
 		(property "Net Z-C" "ZC out"
 			(at 457.2 66.04 0)
@@
 			)
 		)
-		(property "Role" "sensor"
-			(at 396.24 180.34 0)
-			(hide yes)
-			(show_name no)
-			(do_not_autoplace no)
-			(effects
-				(font
-					(size 1.27 1.27)
-				)
-			)
-		)
 		(property "Net Pin_4" "MQ131 out"
 			(at 396.24 180.34 0)
@@
 			)
 		)
-		(property "Role" "bus"
-			(at 248.92 144.78 0)
-			(hide yes)
-			(show_name no)
-			(do_not_autoplace no)
-			(effects
-				(font
-					(size 1.27 1.27)
-				)
-			)
-		)
-		(property "Bus area" "A14:Q18"
-			(at 248.92 144.78 0)
-			(hide yes)
-			(show_name no)
-			(do_not_autoplace no)
-			(effects
-				(font
-					(size 1.27 1.27)
-				)
-			)
-		)
 		(pin "1"
 		)
@@
 			)
 		)
-		(property "Role" "post heavy"
-			(at 391.16 68.58 0)
-			(hide yes)
-			(show_name no)
-			(do_not_autoplace no)
-			(effects
-				(font
-					(size 1.27 1.27)
-				)
-			)
-		)
 		(pin "1"
 		)
@@
 			)
 		)
-		(property "Role" "heavy"
-			(at 261.62 76.2 0)
-			(hide yes)
-			(show_name no)
-			(do_not_autoplace no)
-			(effects
-				(font
-					(size 1.27 1.27)
-				)
-			)
-		)
 		(property "Net Pin_4" "Front fan PWM"
 			(at 261.62 76.2 0)
@@
 			(at 259.08 144.78 0)
 			(hide yes)
-			(show_name no)
-			(do_not_autoplace no)
-			(effects
-				(font
-					(size 1.27 1.27)
-				)
-			)
-		)
-		(property "Role" "bus"
-			(at 259.08 144.78 0)
-			(hide yes)
-			(show_name no)
-			(do_not_autoplace no)
-			(effects
-				(font
-					(size 1.27 1.27)
-				)
-			)
-		)
-		(property "Bus area" "A14:Q18"
-			(at 259.08 144.78 0)
-			(hide yes)

Commit message: finalize kicad standards
Parts:
- A1: Net NRST Reset button -> (none); Net PA0 MQ131 out -> (none); Net PA1 MiCS CO -> (none); Net PA15 I2C SCL -> (none); Net PA5 Front fan tach -> (none); Net PA7 MiCS NO2 -> (none); Net PA8 Front fan PWM -> (none); Net PA9 Rear fan PWM -> (none); Net PB0 ZC in -> (none); Net PB1 TRIAC gate -> (none); Net PB10 Display TX -> (none); Net PB11 Display RX -> (none); Net PB14 Cold-boot button -> (none); Net PB15 Buzzer drive -> (none); Net PB3 Rear fan tach -> (none); Net PB7 I2C SDA -> (none)
- BZ1: Net - Buzzer GND -> (none)
- J5: Net Pin_4 MQ131 out -> (none)
- J6: Net Pin_3 MiCS CO -> (none); Net Pin_4 MiCS NO2 -> (none)
- M2: Net Pin_4 Front fan PWM -> (none)
- M3: Net Pin_4 Rear fan PWM -> (none)
- Q1: Net D Display TX -> (none)
- Q2: Net D Display RX -> (none)
- Q3: Net B Buzzer base -> (none)
- U5: Net Z-C ZC out -> (none)
Connections:
- net MICS_CO_OUT: now reaches J6.3 (Pin_3), R5.2
- net MICS_NO2_OUT: now reaches J6.4 (Pin_4), R7.1
- net FAN_REAR_TACH: now reaches A1.7 (PB3), M3.3 (Pin_3), R22.2
- net DISPLAY_TX: now reaches A1.38 (PB10), Q1.1 (S), R10.2
- net DISPLAY_RX: now reaches A1.39 (PB11), Q2.1 (S), R12.2
- net DISPLAY_RX_5V: now reaches A2.1 (D1/TX), J8.2 (Pin_2), Q2.3 (D), R13.2
- net DISPLAY_TX_5V: now reaches A2.2 (D0/RX), J8.1 (Pin_1), Q1.3 (D), R11.2
- net I2C_SCL: now reaches A1.10 (PA15), J3.3 (Pin_3), J4.3 (SCL), J7.4 (Pin_4), R1.2
- net I2C_SDA: now reaches A1.3 (PB7), J3.2 (Pin_2), J4.4 (SDA), J7.3 (Pin_3), R2.2
- net BOOT_MODE: now reaches A1.18 (PB14), SW2.2
- net ZC_INPUT: now reaches A1.34 (PB0), R14.1, R15.1
- net ZC_OUT: now reaches R14.2, U5.3 (Z-C)
- net FAN_FRONT_TACH: now reaches A1.30 (PA5), M2.3 (Pin_3), R21.2
- net NRST: now reaches A1.24 (NRST), J2.12 (Pin_12), SW1.2
- net MICS_NO2: now reaches A1.32 (PA7), R7.2, R8.1
- net FAN_REAR_PWM_IN: now reaches M3.4 (Pin_4), R20.1
- net FAN_REAR_PWM: now reaches A1.14 (PA9), R20.2
- net FAN_FRONT_PWM_IN: now reaches M2.4 (Pin_4), R19.1
- net FAN_FRONT_PWM: now reaches A1.15 (PA8), R19.2
- net BUZZER_IN: now reaches A1.17 (PB15), R9.1
- net MQ131_ADC: now reaches A1.25 (PA0), R3.2, R4.1
- net MICS_CO1: now reaches A1.26 (PA1), R5.1, R6.1
- net TRIAC_DIMMER: now reaches A1.35 (PB1), U5.4 (PSM)
- net BUZZER_BASE: now reaches Q3.2 (B), R9.2
- net BUZZER_NEG: now reaches BZ1.2 (-), Q3.3 (C)
- net MQ131_OUT: now reaches J5.4 (Pin_4), R3.1
